File: minimalist_shield/nrf24L01Shield.brd (EAGLE design)
At the start: 51.2 x 19.8 mm, 7 parts

Commit message: learned to spell, again.
Other:
- board text added: "http://www.komby.com/rf_shield"
- board text removed: "http://www.komby.com/rf_sheild"
Changed lines of the file:
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@@
 <?xml version="1.0" encoding="utf-8"?>
 <!DOCTYPE eagle SYSTEM "eagle.dtd">
-<eagle version="6.4">
+<eagle version="7.1.0">
 <drawing>
 <settings>
@@
 <text x="3.25" y="1.5" size="1.016" layer="25">SCK</text>
 <text x="34.25" y="4.25" size="0.6096" layer="25">nRF24L01+</text>
-<text x="24.6" y="1.9144" size="1.016" layer="25" align="top-left">http://www.komby.com/rf_sheild</text>
+<text x="24.6" y="1.9144" size="1.016" layer="25" align="top-left">http://www.komby.com/rf_shield</text>
 <text x="40.25" y="6.25" size="0.6096" layer="25" rot="R180">RF Transceiver Sheild</text>
 <text x="40.25" y="6.25" size="0.6096" layer="25" rot="R180">RF Transceiver Sheild</text>
@@
 <pass name="Default">
 <param name="RoutingGrid" value="50mil"/>
+<param name="AutoGrid" value="1"/>
+<param name="Efforts" value="0"/>
+<param name="TopRouterVariant" value="1"/>
 <param name="tpViaShape" value="round"/>
 <param name="PrefDir.1" value="|"/>
