File: minimalist_shield/nrf24L01Shield.sch (EAGLE design)
At the start: 6 parts

Commit message: learned to spell, again.
Other:
- note added: "www.komby.com/rf_shield"
- note removed: "www.komby.com/rf_sheild"
Changed lines of the file:
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@@
 <?xml version="1.0" encoding="utf-8"?>
 <!DOCTYPE eagle SYSTEM "eagle.dtd">
-<eagle version="6.4">
+<eagle version="7.1.0">
 <drawing>
 <settings>
@@
 <plain>
 <text x="165.1" y="-53.34" size="1.778" layer="91">.3</text>
-<text x="81.28" y="-53.34" size="2.54" layer="94">www.komby.com/rf_sheild</text>
+<text x="81.28" y="-53.34" size="2.54" layer="94">www.komby.com/rf_shield</text>
 </plain>
 <instances>
