File: RF1_RS485/RF1_RS485.sch (EAGLE design)
At the start: 9 parts, among them IC1 LTC485N, X1 RJ45-8X

Commit message: updated with new revisions
RF1 RS485 current version, and new Serial board
Parts:
- removed JP2: (no value), jumper:JP8Q
- added PWR, RX, TX: (no value), adafruit:LED3MM
- added R3, R4, R5: 1k, adafruit:R-US_0204/7
- added SV1: (no value), jumper:JP10Q
- added VIN_ENABLE: (no value), jumper:JP1E
- R1, R2: device adafruit:R-US_FLIPFLOP -> adafruit:R-US_0204/7
Connections:
- removed net N$2: JP2.6, JP2.8, X1.2
- removed net N$4: JP2.14, X1.6
- new net DMXB_RENGND2: SV1.20, SV1.4, X1.2
- new net DMXD-_RENGND: SV1.10, SV1.14, X1.1
- new net DMXGND: SV1.16, X1.8
- new net LORGND: SV1.18, X1.6
- new net N$8: R4.1, RX.C
- new net N$9: R5.1, TX.C
- net +5V: now also PWR.A
- net DATA(+)A: now also SV1.11, SV1.7, SV1.9; no longer JP2.1, JP2.9
- net DATA(-)B: now also SV1.1, SV1.3, SV1.5; no longer JP2.11, JP2.5
- net GND: now also R3.2, R4.2, R5.2, SV1.13, SV1.15, SV1.17, SV1.19; no longer JP2.13, JP2.15, JP2.3, JP2.7
- net N$1: now also SV1.6, SV1.8, X1.5; no longer JP2.2, JP2.4, X1.1
- net N$3: now also SV1.12, SV1.2, X1.4; no longer JP2.16, X1.8
- net N$5: now also VIN_ENABLE.1, X1.3; no longer JP2.12, X1.5
- net N$6: now also +V.1, +V.2, VIN_ENABLE.2; no longer JP2.10, X1.4
- net N$7: now also PWR.C, R3.1; no longer +V.1, +V.2, X1.3
- net RX: now also RX.A
- net TX: now also TX.A
Other:
- note added: "DMX 3-4, 9-10, 15-16"
- note added: "LOR 5-6, 11-12, 17-18"
- note added: "REN 1-2, 7-8, 13-14, 19-20"
- note added: "Renard D+ Pin 5 Renard D- Pin 4 Renard GND Pin 1 & 2 LOR D+ Pin 4 LOR D- Pin 5 LOR GND Pin 6 LOR +10VDC Pin 3 DMX D+ Pin 1 DMX D- Pin 2 DMX GND Pin 7 & 8"
- note added: "V0.7"
- note removed: "DMX 1-2, 5-6, 15-16"
- note removed: "LOR 9-10, 11-12, 13-14"
- note removed: "REN 3-4, 7-8, 9-10, 11-12"
- note removed: "V0.5"
- moved on the sheet: +V, X1
